Commit message: Add limits to mimic joints

File: robotiq_description/urdf/robotiq_2f_85_macro.urdf.xacro (robot description, xacro)
@@ -252,4 +252,5 @@
             <axis xyz="0 -1 0" />
             <origin xyz="0.0127 0.0 0.06142" rpy="0 0 0" />
+            <limit lower="0.0" upper="0.8" velocity="0.5" effort="50" />
             <mimic joint="${prefix}robotiq_85_left_knuckle_joint" />
         </joint>
@@ -259,4 +260,5 @@
             <axis xyz="0 -1 0" />
             <origin xyz="-0.0127 0.0 0.06142" rpy="0 0 0" />
+            <limit lower="-0.8" upper="0.0" velocity="0.5" effort="50" />
             <mimic joint="${prefix}robotiq_85_left_knuckle_joint" multiplier="-1" />
         </joint>
@@ -266,4 +268,5 @@
             <axis xyz="0 -1 0" />
             <origin xyz="0.00563134 0.0 0.04718515" rpy="0 0 0" />
+            <limit lower="0.0" upper="0.8" velocity="0.5" effort="50" />
             <mimic joint="${prefix}robotiq_85_left_knuckle_joint" multiplier="-1" />
         </joint>
@@ -273,4 +276,5 @@
             <axis xyz="0 -1 0" />
             <origin xyz="-0.00563134 0.0 0.04718515" rpy="0 0 0" />
+            <limit lower="-0.8" upper="0.0" velocity="0.5" effort="50" />
             <mimic joint="${prefix}robotiq_85_left_knuckle_joint" />
         </joint>
